File: ps2_80_power.kicad_sch (KiCad schematic)
At the start: 309 parts, among them IC1 LM7912_TO220, IC2 SG3524, IC3 LM339, IC4 LM339, IC5 LM339, IC6 TL431P, Q1 MJH16006, Q10 2N4400, Q11 2N4400, Q12 2N4400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

Commit message: a few part value updates
Parts:
- CR38: value 1N75.. -> 1N751 (?)
- R26: value 120 -> 20.0K
- R29: value ? -> 5.36K
Other:
- note added: "2.5V VOLTAGE REFERENCE"
- note added: "5.1V?"
- note added: "VCC UV COMPARATOR"
- note removed: "VOLTAGE REFERENCE"
- moved on the sheet: C20, C25, C28, CR22, CR26, R123, R13, R17, R18, R26, R29
